File: hardware/pcb/TCC-09-05-2026/tcc-16-04-2026-1322.kicad_pcb (KiCad board)
At the start: 2 copper layers, 79 parts, among them J2 Conn_02x20_Odd_Even, J3 Conn_01x10_Pin, J4 Conn_01x10_Pin, SW1 SW_Push, SW10 SW_Push, SW11 SW_Push, SW12 SW_Push, SW13 SW_Push, SW14 SW_Push, SW15 SW_Push, SW16 SW_Push, SW17 SW_Push, SW18 SW_Push, SW19 SW_Push, SW2 SW_Push, SW20 SW_Push, SW21 SW_Push, SW22 SW_Push, SW23 SW_Push, SW24 SW_Push, SW25 SW_Push, SW26 SW_Push, SW27 SW_Push, SW28 SW_Push, SW29 SW_Push, SW3 SW_Push, SW30 SW_Push, SW31 SW_Push, SW32 SW_Push, SW33 SW_Push, SW34 SW_Push, SW35 SW_Push, SW36 SW_Push, SW37 SW_Push, SW38 SW_Push, SW4 SW_Push, SW5 SW_Push, SW6 SW_Push, SW7 SW_Push, SW8 SW_Push, SW9 SW_Push

Commit message: feature/alteracoes-furos-footprint
Parts:
- J3, J4: footprint Connector_PinHeader_2.00mm:PinHeader_2x05_P2.00mm_Vertical -> Connector_PinHeader_2.54mm:PinHeader_2x05_P2.54mm_Vertical
Routing:
- net Col1: track 308.7 -> 371.3 mm, vias 1 -> 3
- net Row4: track 294.1 -> 289.6 mm, vias 4 -> 2
- net Col2: track 242.6 -> 245.4 mm, vias 1 -> 3
- net Col0: track 347.3 -> 344.7 mm, vias 3 -> 1
- net Row5: track 319.8 -> 321.0 mm, vias 2 -> 0
- net Row2: track 248.1 -> 247.1 mm, vias 2 -> 0
- net Row0: track 368.3 -> 367.5 mm, vias 2 -> 0
- net Row3: track 290.7 -> 290.0 mm, vias 4 -> 2
- net Row1: track 280.4 -> 280.0 mm, vias 2 -> 0
Other:
- board outline added: 191.6 x 128.9 mm
