File: hardware/pcb/TCC-06-17-2026-PTH - Copy/Placa/Placa.kicad_pcb (KiCad board)
At the start: 2 copper layers, 196.5 x 125.4 mm, 81 parts, among them J1 Conn_01x03, J3 Conn_01x02, J6 Conn_01x03, J7 Conn_01x03, J8 Conn_01x02, SW1 SW_Push, SW10 SW_Push, SW11 SW_Push, SW12 SW_Push, SW13 SW_Push, SW14 SW_Push, SW15 SW_Push, SW16 SW_Push, SW17 SW_Push, SW18 SW_Push, SW19 SW_Push, SW2 SW_Push, SW20 SW_Push, SW21 SW_Push, SW22 SW_Push, SW23 SW_Push, SW24 SW_Push, SW25 SW_Push, SW26 SW_Push, SW27 SW_Push, SW28 SW_Push, SW29 SW_Push, SW3 SW_Push, SW30 SW_Push, SW31 SW_Push, SW32 SW_Push, SW33 SW_Push, SW34 SW_Push, SW35 SW_Push, SW36 SW_Push, SW37 SW_Push, SW38 SW_Push, SW4 SW_Push, SW5 SW_Push, SW6 SW_Push, SW7 SW_Push, SW8 SW_Push, SW9 SW_Push

Commit message: Ajustes na pcb
Parts:
- J1, J3, J6, J7, J8: moved to B.Cu
- moved J1 5.10 mm to (94.0, 151.1), turned to 180 degrees
- moved J7 5.09 mm to (205.8, 151.2), turned to 180 degrees
- moved J6 4.95 mm to (218.8, 151.0), turned to 180 degrees
- moved J8 2.70 mm to (175.0, 151.1), turned to 180 degrees
- moved J3 0.70 mm to (159.5, 151.1), turned to 180 degrees
Connections:
- J1 pad 1: Col0 -> Col2
- J1 pad 3: Col2 -> Col0
- J3 pad 1: Col3 -> Col4
- J3 pad 2: Col4 -> Col3
- J6 pad 1: Row2 -> Row0
- J6 pad 3: Row0 -> Row2
- J7 pad 1: Row5 -> Row3
- J7 pad 3: Row3 -> Row5
- J8 pad 1: Col5 -> Col6
- J8 pad 2: Col6 -> Col5
Routing:
- net Col3: track 194.9 -> 191.7 mm, vias 0 -> 1
- net Col4: track 158.6 -> 161.5 mm, vias 0 -> 1
- net Row3: track 237.6 -> 239.2 mm, vias 1 -> 0
- net Col5: track 167.3 -> 167.9 mm, vias 0 -> 1
- net Col1: track 198.0 -> 198.2 mm, vias 0 -> 1
- net Col6: track 189.5 -> 189.3 mm, vias 0 -> 1
- net Row5: track 231.7 -> 231.8 mm, vias 1 -> 0
- net Row2: track 271.5 -> 271.4 mm, vias 1 -> 0
- net Col2: track 159.8 -> 159.7 mm, vias 0 -> 1
- net Row4: track 236.2 -> 236.3 mm, vias 1 -> 0
- net Row1: vias 1 -> 0
- net Row0: vias 1 -> 0
- net Col0: vias 0 -> 1

Commit message: refactor(pcb): reorganiza posicionamento dos componentes
Parts:
- moved J7 4.40 mm to (201.3, 151.2)
Routing:
- net Row5: track 231.8 -> 227.4 mm
- net Row3: track 239.2 -> 242.0 mm
- net Row4: track 236.3 -> 238.1 mm
